File: circuits/module_generic_top_board/module_generic_top_board.kicad_pcb (KiCad board)
At the start: 2 copper layers, 24.1 x 77.5 mm, 16 parts, among them P1 CONN_01X08, P2 CONN_01X08, P3 CONN_01X03, P4 CONN_01X08, P5 CONN_01X02, P6 CONN_01X11, P7 CONN_01X01, P8 CONN_01X01, U1 4051, U2 74HC595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

Commit message: Update Module Generic Top Board
Parts:
- removed RR1: RR8, Resistors_ThroughHole:Resistor_Array_SIP8
- added RN1: 10K, Resistors_THT:R_Array_SIP9, F.Cu at (146.7, 143.5)
- moved P3 0.64 mm to (134.6, 114.9)
Routing:
- net GND: track 215.6 -> 216.2 mm
- net Net-(P3-Pad3): track 26.9 -> 27.5 mm
