File: circuits/teensy_mother_board/teensy_mother_board.kicad_pcb (KiCad board)
At the start: 2 copper layers, 64.8 x 45.7 mm, 13 parts, among them P1 CONN_01X01, P10 CONN_01X02, P11 CONN_01X02, P12 CONN_01X02, P13 CONN_01X02, P2 CONN_01X01, P3 CONN_01X01, P4 CONN_01X01, P5 CONN_02X05, P6 CONN_02X03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

Commit message: Update circuits
Routing:
- net /MASTER_MUX_B: track 67.6 -> 56.2 mm
- net /MASTER_MUX_C: track 49.6 -> 48.4 mm
Other:
- net class Default: via_dia 0.6 -> 1; via_drill 0.4 -> 0.5
Changed lines of the file:
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@@
-(kicad_pcb (version 4) (host pcbnew 4.0.2+dfsg1-2~bpo8+1-stable)
+(kicad_pcb (version 4) (host pcbnew 4.0.6+dfsg1-1)
   (general
     (links 31)
     (no_connects 0)
-    (area 93.951667 87.267 163.858334 135.849)
+    (area 94.026667 87.417 163.783334 135.949)
     (thickness 1.6)
     (drawings 5)
@@
   (title_block
     (title "Teensy Mother Board")
+    (date 2017-11-01)
+    (rev 1)
     (company "Alexandros Drymonitis")
   )
@@
     (segment_width 0.2)
     (edge_width 0.15)
-    (via_size 0.6)
-    (via_drill 0.4)
+    (via_size 1)
+    (via_drill 0.5)
     (via_min_size 0.5)
     (via_min_drill 0.3)
@@
     (clearance 0.2)
     (trace_width 0.3)
-    (via_dia 0.6)
-    (via_drill 0.4)
+    (via_dia 1)
+    (via_drill 0.5)
     (uvia_dia 0.3)
     (uvia_drill 0.1)
@@
       (net 10 /MOSI))
   )
-  (gr_text "© Alexandros Drymonitis" (at 109.22 92.075) (layer B.Cu)
-    (effects (font (size 0.762 0.762) (thickness 0.1905)) (justify mirror))
+  (gr_text "© Alexandros Drymonitis" (at 111.125 91.44) (layer B.Cu)
+    (effects (font (size 1 1) (thickness 0.1905)) (justify mirror))
   )
   (gr_line (start 96.52 134.62) (end 96.52 88.9) (angle 90) (layer Edge.Cuts) (width 0.15))
@@
   (gr_line (start 161.29 88.9) (end 161.29 134.62) (angle 90) (layer Edge.Cuts) (width 0.15))
   (gr_line (start 96.52 88.9) (end 161.29 88.9) (angle 90) (layer Edge.Cuts) (width 0.15))
+  (segment (start 151.13 121.92) (end 148.59 121.92) (width 0.3) (layer B.Cu) (net 1))
+  (via (at 148.59 132.08) (size 1) (drill 0.5) (layers F.Cu B.Cu) (net 1))
+  (segment (start 148.59 121.92) (end 148.59 132.08) (width 0.3) (layer F.Cu) (net 1))
+  (via (at 148.59 121.92) (size 1) (drill 0.5) (layers F.Cu B.Cu) (net 1))
   (segment (start 100.33 110.49) (end 106.68 110.49) (width 0.3) (layer B.Cu) (net 1) (status 10))
   (segment (start 106.68 110.49) (end 113.03 116.84) (width 0.3) (layer B.Cu) (net 1))
@@
   (segment (start 158.75 132.08) (end 148.59 132.08) (width 0.3) (layer B.Cu) (net 1))
   (segment (start 99.06 132.08) (end 113.03 132.08) (width 0.3) (layer B.Cu) (net 1))
-  (segment (start 151.13 121.92) (end 148.59 121.92) (width 0.3) (layer B.Cu) (net 1))
   (segment (start 113.03 132.08) (end 113.03 124.46) (width 0.3) (layer B.Cu) (net 1))
   (segment (start 148.59 132.08) (end 124.46 132.08) (width 0.3) (layer B.Cu) (net 1))
   (segment (start 124.46 132.08) (end 113.03 132.08) (width 0.3) (layer B.Cu) (net 1))
-  (via (at 148.59 132.08) (size 0.6) (drill 0.4) (layers F.Cu B.Cu) (net 1))
-  (segment (start 148.59 121.92) (end 148.59 132.08) (width 0.3) (layer F.Cu) (net 1))
-  (via (at 148.59 121.92) (size 0.6) (drill 0.4) (layers F.Cu B.Cu) (net 1))
   (segment (start 158.75 108.585) (end 160.02 109.855) (width 0.3) (layer B.Cu) (net 1))
   (segment (start 151.13 111.76) (end 151.13 110.49) (width 0.3) (layer B.Cu) (net 2))
@@
   (segment (start 153.67 125.73) (end 152.4 127) (width 0.3) (layer B.Cu) (net 10))
   (segment (start 134.62 97.79) (end 134.62 100.33) (width 0.3) (layer B.Cu) (net 11))
-  (segment (start 119.38 100.33) (end 119.38 99.06) (width 0.3) (layer B.Cu) (net 11))
-  (via (at 119.38 100.33) (size 0.6) (drill 0.4) (layers F.Cu B.Cu) (net 11))
+  (via (at 119.38 100.33) (size 1) (drill 0.5) (layers F.Cu B.Cu) (net 11))
   (segment (start 134.62 100.33) (end 119.38 100.33) (width 0.3) (layer F.Cu) (net 11))
-  (via (at 134.62 100.33) (size 0.6) (drill 0.4) (layers F.Cu B.Cu) (net 11))
+  (via (at 134.62 100.33) (size 1) (drill 0.5) (layers F.Cu B.Cu) (net 11))
   (segment (start 119.38 99.06) (end 120.65 97.79) (width 0.3) (layer B.Cu) (net 11))
   (segment (start 123.19 124.46) (end 123.19 119.38) (width 0.3) (layer B.Cu) (net 11))
   (segment (start 119.38 99.06) (end 120.65 97.79) (width 0.3) (layer B.Cu) (net 11))
-  (segment (start 119.38 115.57) (end 119.38 99.06) (width 0.3) (layer B.Cu) (net 11))
+  (segment (start 119.38 115.57) (end 119.38 100.33) (width 0.3) (layer B.Cu) (net 11))
+  (segment (start 119.38 100.33) (end 119.38 99.06) (width 0.3) (layer B.Cu) (net 11))
   (segment (start 123.19 119.38) (end 119.38 115.57) (width 0.3) (layer B.Cu) (net 11))
   (segment (start 120.65 95.25) (end 120.65 92.71) (width 0.3) (layer B.Cu) (net 12))
@@
   (segment (start 143.51 109.22) (end 143.51 108.585) (width 0.3) (layer B.Cu) (net 13))
   (segment (start 139.7 97.79) (end 139.7 102.87) (width 0.3) (layer B.Cu) (net 14))
-  (segment (start 127 102.87) (end 127 114.3) (width 0.3) (layer B.Cu) (net 14))
-  (via (at 127 102.87) (size 0.6) (drill 0.4) (layers F.Cu B.Cu) (net 14))
+  (via (at 127 102.87) (size 1) (drill 0.5) (layers F.Cu B.Cu) (net 14))
   (segment (start 139.7 102.87) (end 127 102.87) (width 0.3) (layer F.Cu) (net 14))
-  (via (at 139.7 102.87) (size 0.6) (drill 0.4) (layers F.Cu B.Cu) (net 14))
+  (via (at 139.7 102.87) (size 1) (drill 0.5) (layers F.Cu B.Cu) (net 14))
   (segment (start 127 114.3) (end 125.73 115.57) (width 0.3) (layer B.Cu) (net 14))
   (segment (start 125.73 115.57) (end 125.73 124.46) (width 0.3) (layer B.Cu) (net 14))
   (segment (start 125.73 124.46) (end 125.73 115.57) (width 0.3) (layer B.Cu) (net 14))
   (segment (start 127 99.06) (end 125.73 97.79) (width 0.3) (layer B.Cu) (net 14))
-  (segment (start 127 114.3) (end 127 99.06) (width 0.3) (layer B.Cu) (net 14))
+  (segment (start 127 114.3) (end 127 102.87) (width 0.3) (layer B.Cu) (net 14))
+  (segment (start 127 102.87) (end 127 99.06) (width 0.3) (layer B.Cu) (net 14))
   (segment (start 125.73 115.57) (end 127 114.3) (width 0.3) (layer B.Cu) (net 14))
   (segment (start 139.7 95.25) (end 139.7 93.98) (width 0.3) (layer B.Cu) (net 15))
@@
     (polygon
       (pts
-        (xy 161.29 134.62) (xy 96.52 134.62) (xy 96.52 88.9) (xy 161.29 88.9) (xy 161.29 134.62)
+        (xy 161.29 134.62) (xy 96.52 134.62) (xy 96.52 88.9) (xy 161.29 88.9)
       )
     )
